File: Audio-Path/Audio-Path.kicad_sch (KiCad schematic)
At the start: 52 parts, among them IC252 BA15218, IC253 BA15218, J5012 L, J5013 R_SW

Commit message: Redo filter response
Parts:
- IC252, IC253: value BA15218 -> BA15218F; symbol Device:Opamp_Dual -> loopy-parts:BA15218F
Other:
- note added: "-14dB/oct"
- note added: "-20dB"
- note added: "-40dB"
- note added: "0dB"
- note added: "100KHz"
- note added: "10KHz"
- note added: "1K +0.1dB"
- note added: "1KHz"
- note added: "7.5K +4.8dB"
- note added: "85K -43dB"
- note added: "Based on data from http://sim.okawa-denshi.jp/en/Sallen3tool.php"
- note added: "Gain 1.0x"
- note added: "Gain 6.8x"
- note added: "Theoretical frequency response"
- note added: "fs = 84864Hz"
- note added: "~10.5K 0dB"
- note removed: "1KHz +0.1dB"
- note removed: "7.5KHz +4.8dB"
- note removed: "85KHz -43dB"
- note removed: "Gain ~1.0x"
- note removed: "Gain ~6.8x"
- note removed: "THEORETICAL"
- note removed: "~10.6KHz 0dB"
Changed lines of the file:
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@@
 	(generator_version "9.0")
 	(paper "A4")
-	(bezier
-		(pts
-			(xy 90.17 69.85) (xy 91.44 71.12) (xy 93.98 76.2) (xy 96.52 82.55)
+	(rectangle
+		(start 130.81 130.81)
+		(end 138.43 133.35)
+		(stroke
+			(width 0)
+			(type default)
+		)
+		(fill
+			(type none)
 		)
+	)
+	(rectangle
+		(start 95.25 130.81)
+		(end 102.87 133.35)
 		(stroke
 			(width 0)
@@
 	(bezier
 		(pts
-			(xy 81.28 69.85) (xy 86.36 69.85) (xy 87.63 67.31) (xy 90.17 69.85)
+			(xy 88.9 71.12) (xy 91.44 73.66) (xy 100.33 78.74) (xy 102.87 81.28)
 		)
 		(stroke
-			(width 0)
+			(width 0.254)
 			(type solid)
 		)
@@
 		)
 	)
-	(text "~10.6KHz 0dB"
+	(bezier
+		(pts
+			(xy 74.93 71.12) (xy 87.63 71.12) (xy 86.36 68.58) (xy 88.9 71.12)
+		)
+		(stroke
+			(width 0.254)
+			(type solid)
+		)
+		(fill
+			(type none)
+		)
+	)
+	(text "~10.5K 0dB"
 		(exclude_from_sim no)
-		(at 90.17 72.39 0)
+		(at 88.9 73.66 0)
 		(effects
 			(font
@@
 		)
 	)
-	(text "THEORETICAL"
+	(text "fs = 84864Hz"
 		(exclude_from_sim no)
-		(at 107.95 71.12 0)
+		(at 35.56 38.1 0)
 		(effects
 			(font
@@
 		)
 	)
+	(text "Based on data from http://sim.okawa-denshi.jp/en/Sallen3tool.php"
+		(exclude_from_sim no)
+		(at 63.5 83.82 0)
+		(effects
+			(font
+				(size 0.762 0.762)
+			)
+			(justify left top)
+		)
+	)
+	(text "Theoretical frequency response"
+		(exclude_from_sim no)
+		(at 63.5 63.5 0)
+		(effects
+			(font
+				(size 1.27 1.27)
+			)
+			(justify left top)
+		)
+	)
+	(text "10KHz"
+		(exclude_from_sim no)
+		(at 88.9 82.55 0)
+		(effects
+			(font
+				(size 0.762 0.762)
+			)
+		)
+	)
 	(text "Input Coupling"
 		(exclude_from_sim no)
@@
 		)
 	)
-	(text "1KHz +0.1dB"
+	(text "100KHz"
 		(exclude_from_sim no)
-		(at 73.66 67.31 0)
+		(at 102.87 82.55 0)
+		(effects
+			(font
+				(size 0.762 0.762)
+			)
+		)
+	)
+	(text "1KHz"
+		(exclude_from_sim no)
+		(at 74.93 82.55 0)
+		(effects
+			(font
+				(size 0.762 0.762)
+			)
+		)
+	)
+	(text "1K +0.1dB"
+		(exclude_from_sim no)
+		(at 74.93 68.58 0)
 		(effects
 			(font
@@
 		)
 	)
+	(text "-20dB"
+		(exclude_from_sim no)
+		(at 67.31 75.565 0)
+		(effects
+			(font
+				(size 0.762 0.762)
+			)
+			(justify right)
+		)
+	)
 	(text "~300kHz LPF"
 		(exclude_from_sim no)
@@
 		)
 	)
+	(text "-14dB/oct"
+		(exclude_from_sim no)
+		(at 93.98 77.47 0)
+		(effects
+			(font
+				(size 1.27 1.27)
+			)
+			(justify right top)
+		)
+	)
 	(text "Virtual ground"
 		(exclude_from_sim no)
@@
 		)
 	)
-	(text "7.5KHz +4.8dB"
+	(text "0dB"
 		(exclude_from_sim no)
-		(at 87.63 66.04 0)
+		(at 67.31 71.12 0)
+		(effects
+			(font
+				(size 0.762 0.762)
+			)
+			(justify right)
+		)
+	)
+	(text "7.5K +4.8dB"
+		(exclude_from_sim no)
+		(at 86.36 68.58 0)
 		(effects
 			(font
@@
 		)
 	)
-	(text "Gain ~6.8x"
+	(text "Gain 6.8x"
 		(exclude_from_sim no)
 		(at 113.03 33.02 0)
@@
 		)
 	)
-	(text "Gain ~1.0x"
+	(text "Gain 1.0x"
 		(exclude_from_sim no)
 		(at 113.03 64.77 0)
@@
 		)
 	)
+	(text "-40dB"
+		(exclude_from_sim no)
+		(at 67.31 80.01 0)
+		(effects
+			(font
+				(size 0.762 0.762)
+			)
+			(justify right)
+		)
+	)
 	(text "AV Receiver"
 		(exclude_from_sim no)
@@
 	(text "Polarized caps in audio path should be electrolytic >= 10uF"
 		(exclude_from_sim no)
-		(at 63.5 139.7 0)
+		(at 60.96 139.7 0)
 		(effects
 			(font
@@
 		)
 	)
-	(text "85KHz -43dB"
+	(text "85K\n-43dB"
 		(exclude_from_sim no)
-		(at 93.98 80.01 0)
+		(at 101.6 77.47 0)
 		(effects
 			(font
 				(size 1.27 1.27)
 			)
-			(justify right)
+			(justify bottom)
 		)
 	)
@@
 	(polyline
 		(pts
-			(xy 66.04 82.55) (xy 99.06 82.55)
+			(xy 67.31 81.28) (xy 105.41 81.28)
 		)
 		(stroke
@@
 	(polyline
 		(pts
-			(xy 66.04 69.85) (xy 81.28 69.85)
+			(xy 67.31 71.12) (xy 74.93 71.12)
 		)
 		(stroke
-			(width 0)
+			(width 0.254)
 			(type solid)
 		)
@@
 		)
 	)
+	(polyline
+		(pts
+			(xy 101.6 80.01) (xy 101.6 77.47)
+		)
+		(stroke
+			(width 0)
+			(type default)
+		)
+	)
 	(wire
 		(pts
@@
 		)
 	)
-	(polyline
-		(pts
-			(xy 81.28 69.85) (xy 81.28 69.85)
-		)
-		(stroke
-			(width 0)
-			(type solid)
-		)
-	)
 	(wire
 		(pts
@@
 	(polyline
 		(pts
-			(xy 66.04 66.04) (xy 66.04 82.55)
+			(xy 67.31 67.31) (xy 67.31 81.28)
 		)
 		(stroke
@@
 	(polyline
 		(pts
-			(xy 73.66 67.31) (xy 73.66 68.58)
+			(xy 74.93 68.58) (xy 74.93 71.12)
 		)
 		(stroke
@@
 	(polyline
 		(pts
-			(xy 90.17 72.39) (xy 90.17 71.12)
+			(xy 88.9 73.025) (xy 88.9 71.12)
 		)
 		(stroke
@@
 		)
 	)
+	(polyline
+		(pts
+			(xy 94.615 77.47) (xy 95.885 76.2)
+		)
+		(stroke
+			(width 0)
+			(type default)
+		)
+	)
 	(wire
 		(pts
@@
 	(polyline
 		(pts
-			(xy 87.63 66.04) (xy 87.63 67.31)
+			(xy 86.995 68.58) (xy 86.995 69.85)
 		)
 		(stroke
@@
 	)
 	(symbol
-		(lib_id "Device:Opamp_Dual")
+		(lib_id "loopy-parts:BA15218F")
 		(at 99.06 38.1 0)
 		(mirror x)
@@
 			)
 		)
-		(property "Value" "BA15218"
+		(property "Value" "BA15218F"
 			(at 100.33 45.72 0)
 			(effects
@@
 					(size 1.27 1.27)
 				)
+				(hide yes)
 			)
 		)
@@
 	)
 	(symbol
-		(lib_id "Device:Opamp_Dual")
+		(lib_id "loopy-parts:BA15218F")
 		(at 134.62 134.62 90)
 		(mirror x)
@@
 			)
 		)
-		(property "Value" "BA15218"
+		(property "Value" "BA15218F"
 			(at 134.62 129.54 90)
 			(effects
@@
 					(size 1.27 1.27)
 				)
+				(hide yes)
 			)
 		)
@@
 	)
 	(symbol
-		(lib_id "Device:Opamp_Dual")
+		(lib_id "loopy-parts:BA15218F")
 		(at 99.06 134.62 90)
 		(mirror x)
@@
 			)
 		)
-		(property "Value" "BA15218"
+		(property "Value" "BA15218F"
 			(at 99.06 129.54 90)
 			(effects
@@
 					(size 1.27 1.27)
 				)
+				(hide yes)
 			)
 		)
@@
 	)
 	(symbol
-		(lib_id "Device:Opamp_Dual")
+		(lib_id "loopy-parts:BA15218F")
 		(at 99.06 96.52 0)
 		(mirror x)
@@
 			)
 		)
-		(property "Value" "BA15218"
+		(property "Value" "BA15218F"
 			(at 100.33 104.14 0)
 			(effects
@@
 					(size 1.27 1.27)
 				)
+				(hide yes)
 			)
 		)
@@
 	)
 	(symbol
-		(lib_id "Device:Opamp_Dual")
+		(lib_id "loopy-parts:BA15218F")
 		(at 134.62 40.64 0)
 		(mirror x)
@@
 			)
 		)
-		(property "Value" "BA15218"
+		(property "Value" "BA15218F"
 			(at 134.62 49.53 0)
 			(effects
@@
 					(size 1.27 1.27)
 				)
+				(hide yes)
 			)
 		)
@@
 	)
 	(symbol
-		(lib_id "Device:Opamp_Dual")
+		(lib_id "loopy-parts:BA15218F")
 		(at 134.62 93.98 0)
 		(unit 2)
@@
 		(fields_autoplaced yes)
 		(property "Reference" "IC253"
-			(at 134.62 85.09 0)
+			(at 134.62 83.82 0)
 			(effects
 				(font
@@
 			)
 		)
-		(property "Value" "BA15218"
-			(at 134.62 87.63 0)
+		(property "Value" "BA15218F"
+			(at 134.62 86.36 0)
 			(effects
 				(font
@@
 					(size 1.27 1.27)
 				)
+				(hide yes)
 			)
 		)
