File: Gamepad/Gamepad.kicad_sch (KiCad schematic)
At the start: 32 parts, among them J1 Cable connector, J2 Controller Plug

Commit message: Update all to Kicad 9.0 and cleanup
Connections:
- net ROW0 renamed OUT0
- net ROW1 renamed OUT1
- net ROW2 renamed OUT2
- net data0 renamed IN0
- net data1 renamed IN1
- net data2 renamed IN2
- net data3 renamed IN3
Other:
- note added: "Detect"
- note added: "IN0"
- note added: "IN1"
- note added: "IN2"
- note added: "IN3"
- note added: "IN4"
- note added: "IN5"
- note added: "IN6"
- note added: "IN7"
- note added: "OUT0"
- note added: "OUT1"
- note added: "OUT2"
- note added: "OUT3"
- note added: "OUT4"
- note added: "OUT5"
- note removed: "Presence"
- note removed: "ROW0"
- note removed: "ROW1"
- note removed: "ROW2"
- note removed: "ROW3"
- note removed: "ROW4"
- note removed: "ROW5"
- note removed: "data0"
- note removed: "data1"
- note removed: "data2"
- note removed: "data3"
- note removed: "data4"
- note removed: "data5"
- note removed: "data6"
- note removed: "data7"
- moved on the sheet: J1, J2, JH
